File: hyperion.kicad_sch (KiCad schematic)
At the start: 30 parts, among them J1 AudioJack3, Q1 NPN, Q2 NPN, Q3 PNP, SW1 SW_Slide_DPDT, SW2 Neck, SW3 Bridge, SW4 Strangle

Commit message: correct the guitar wiring in the schematic
Connections:
- net at J1.T, SW1.2 (B): no longer RV2.2
- net at RV1.1, SW1.5 (B), SW2.1 (A)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: now also RV2.2
- net at SW1.3 (C): now also SW1.4 (A)
Changed lines of the file:
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@@
 	)
 	(junction
-		(at 229.87 114.3)
+		(at 222.25 93.98)
 		(diameter 0)
 		(color 0 0 0 0)
@@
 	(wire
 		(pts
+			(xy 222.25 93.98) (xy 184.15 93.98)
+		)
+		(stroke
+			(width 0)
+			(type default)
+		)
+	)
+	(wire
+		(pts
+			(xy 229.87 124.46) (xy 229.87 114.3)
+		)
+		(stroke
+			(width 0)
+			(type default)
+		)
+	)
+	(wire
+		(pts
 			(xy 234.95 146.05) (xy 234.95 147.32)
 		)
@@
 	(wire
 		(pts
+			(xy 229.87 114.3) (xy 240.03 114.3)
+		)
+		(stroke
+			(width 0)
+			(type default)
+		)
+	)
+	(wire
+		(pts
 			(xy 195.58 127) (xy 222.25 127)
 		)
@@
 	(wire
 		(pts
-			(xy 229.87 114.3) (xy 229.87 124.46)
-		)
-		(stroke
-			(width 0)
-			(type default)
-		)
-	)
-	(wire
-		(pts
 			(xy 105.41 109.22) (xy 113.03 109.22)
 		)
@@
 	(wire
 		(pts
+			(xy 240.03 119.38) (xy 240.03 121.92)
+		)
+		(stroke
+			(width 0)
+			(type default)
+		)
+	)
+	(wire
+		(pts
 			(xy 128.27 116.84) (xy 128.27 109.22)
 		)
@@
 	(wire
 		(pts
-			(xy 222.25 114.3) (xy 229.87 114.3)
-		)
-		(stroke
-			(width 0)
-			(type default)
-		)
-	)
-	(wire
-		(pts
 			(xy 110.49 116.84) (xy 113.03 116.84)
 		)
@@
 	(wire
 		(pts
-			(xy 240.03 114.3) (xy 229.87 114.3)
-		)
-		(stroke
-			(width 0)
-			(type default)
-		)
-	)
-	(wire
-		(pts
-			(xy 262.89 93.98) (xy 184.15 93.98)
+			(xy 250.19 121.92) (xy 240.03 121.92)
+		)
+		(stroke
+			(width 0)
+			(type default)
+		)
+	)
+	(wire
+		(pts
+			(xy 262.89 93.98) (xy 222.25 93.98)
 		)
 		(stroke
@@
 	(wire
 		(pts
+			(xy 250.19 119.38) (xy 250.19 121.92)
+		)
+		(stroke
+			(width 0)
+			(type default)
+		)
+	)
+	(wire
+		(pts
 			(xy 144.78 110.49) (xy 144.78 116.84)
 		)
@@
 	(wire
 		(pts
-			(xy 222.25 127) (xy 222.25 114.3)
-		)
-		(stroke
+			(xy 222.25 93.98) (xy 222.25 127)
+		)
+		(stroke
